Commit message: feat(model): Add omni three-wheel drive configuration

File: src/robot_description/urdf/xlerobot/meshes/xlerobot/assets/xlerobot.urdf (robot description, URDF)
Before this commit: robot xlerobot, 56 links, 55 joints
Links:
- removed link wheel_1
- removed link wheel_1_hub
- removed link wheel_1_motor
- removed link wheel_1_mount
- removed link wheel_2
- removed link wheel_2_hub
- removed link wheel_2_motor
- removed link wheel_2_mount
- removed link wheel_3
- removed link wheel_3_hub
- removed link wheel_3_motor
- removed link wheel_3_mount
- removed link wheel_base_plate
- added link left_wheel, mass 1; collision cylinder length=0.04 radius=0.05
- added link right_wheel, mass 1; collision cylinder length=0.04 radius=0.05
Joints:
- removed joint ST3215_Servo_Motor-v1-1_Hub-2---Servo
- removed joint ST3215_Servo_Motor-v1-2_Hub---Servo
- removed joint ST3215_Servo_Motor-v1_Revolute-40
- removed joint wheel_1_motor_fixed
- removed joint wheel_1_mount_fixed
- removed joint wheel_1_wheel_fixed
- removed joint wheel_2_motor_fixed
- removed joint wheel_2_mount_fixed
- removed joint wheel_2_wheel_fixed
- removed joint wheel_3_motor_fixed
- removed joint wheel_3_mount_fixed
- removed joint wheel_3_wheel_fixed
- removed joint wheel_base_plate_fixed
- added joint left_wheel_joint: type continuous, parent chassis, child left_wheel, origin xyz=-0.15 0.225 -0.32 rpy=1.5707963 0 3.1415927, axis 0 0 1, limit effort=0 velocity=0
- added joint right_wheel_joint: type continuous, parent chassis, child right_wheel, origin xyz=-0.15 -0.225 -0.32 rpy=1.5707963 0 3.1415927, axis 0 0 1, limit effort=0 velocity=0
