Commit message: feat(simulation): add XLeRobot MuJoCo simulation and RViz joint state sync

File: src/robot_description/urdf/xlerobot/xlerobot.urdf (robot description, URDF)
Before this commit: robot xlerobot, 45 links, 44 joints
Links:
- link world: mass 0 -> None
Joints:
- joint joint_0: type floating -> fixed

Commit message: feat(wheel model): switch omni base to parallel differential drive

File: src/robot_description/urdf/xlerobot/xlerobot.urdf (robot description, URDF)
Before this commit: robot xlerobot, 56 links, 55 joints
Links:
- removed link wheel_1
- removed link wheel_1_hub
- removed link wheel_1_motor
- removed link wheel_1_mount
- removed link wheel_2
- removed link wheel_2_hub
- removed link wheel_2_motor
- removed link wheel_2_mount
- removed link wheel_3
- removed link wheel_3_hub
- removed link wheel_3_motor
- removed link wheel_3_mount
- added link left_wheel, mass 1.3542854082; visual mesh filename=package://robot_description/urdf/xlerobot/meshes/xlerobot/a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 scale=0.001 0.001 0.001
- added link left_wheel_hub, mass 0.0866549611; visual mesh filename=package://robot_description/urdf/xlerobot/meshes/xlerobot/a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 scale=0.001 0.001 0.001
- added link left_wheel_motor, mass 0.06589629619; visual mesh filename=package://robot_description/urdf/xlerobot/meshes/xlerobot/a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 scale=0.001 0.001 0.001
- added link left_wheel_mount, mass 0.03588401719; visual mesh filename=package://robot_description/urdf/xlerobot/meshes/xlerobot/a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 scale=0.001 0.001 0.001
- added link right_wheel, mass 1.3542854082; visual mesh filename=package://robot_description/urdf/xlerobot/meshes/xlerobot/a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 scale=0.001 0.001 0.001
- added link right_wheel_hub, mass 0.0866549611; visual mesh filename=package://robot_description/urdf/xlerobot/meshes/xlerobot/a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 scale=0.001 0.001 0.001
- added link right_wheel_motor, mass 0.06589629619; visual mesh filename=package://robot_description/urdf/xlerobot/meshes/xlerobot/a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 scale=0.001 0.001 0.001
- added link right_wheel_mount, mass 0.03588401719; visual mesh filename=package://robot_description/urdf/xlerobot/meshes/xlerobot/a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 scale=0.001 0.001 0.001
Joints:
- removed joint ST3215_Servo_Motor-v1_Revolute-40
- removed joint wheel_1_motor_fixed
- removed joint wheel_1_mount_fixed
- removed joint wheel_1_wheel_fixed
- removed joint wheel_2_motor_fixed
- removed joint wheel_2_mount_fixed
- removed joint wheel_2_wheel_fixed
- removed joint wheel_3_motor_fixed
- removed joint wheel_3_mount_fixed
- removed joint wheel_3_wheel_fixed
- added joint left_wheel_fixed: type fixed, parent left_wheel_hub, child left_wheel, origin xyz=0 0 0.01905 rpy=-3.1415926536 0 -0.2617993878
- added joint left_wheel_motor_fixed: type fixed, parent left_wheel_mount, child left_wheel_motor, origin xyz=0.0096 -0.00489 0.01436 rpy=0 0 -1.5707963268
- added joint left_wheel_mount_fixed: type fixed, parent chassis, child left_wheel_mount, origin xyz=-0.12939 0.18675 -0.34356 rpy=0 0 1.5707963268
- added joint right_wheel_fixed: type fixed, parent right_wheel_hub, child right_wheel, origin xyz=0 0 0.019049822 rpy=3.1415926536 0 1.8325957146
- added joint right_wheel_motor_fixed: type fixed, parent right_wheel_mount, child right_wheel_motor, origin xyz=0.0104 -0.00489 0.01436 rpy=0 0 -1.5707963268
- added joint right_wheel_mount_fixed: type fixed, parent chassis, child right_wheel_mount, origin xyz=-0.129390007876 -0.264050004161 -0.34356 rpy=0 0 1.5707963268
- joint ST3215_Servo_Motor-v1-1_Hub-2---Servo: child wheel_2_hub -> right_wheel_hub; origin xyz=-0.0254998972 0.0096001780 0 rpy=-1.5707963268 0 0 -> xyz=-0.0254998972 0.009600178 0 rpy=-1.5707963268 0 0; parent wheel_2_motor -> right_wheel_motor
- joint ST3215_Servo_Motor-v1-2_Hub---Servo: child wheel_1_hub -> left_wheel_hub; origin xyz=-0.0255 0.012775 0 rpy=-1.5707963268 0 3.1415926536 -> xyz=-0.0255 0.0096 0 rpy=-1.5707963268 0 3.1415926536; parent wheel_1_motor -> left_wheel_motor

Commit message: feat(robot): replace omni wheel assembly with differential-drive wheels

File: src/robot_description/urdf/xlerobot/xlerobot.urdf (robot description, URDF)
Before this commit: robot xlerobot, 52 links, 51 joints
Links:
- removed link left_wheel_hub
- removed link left_wheel_motor
- removed link left_wheel_mount
- removed link right_wheel_hub
- removed link right_wheel_motor
- removed link right_wheel_mount
- removed link wheel_base_plate
- link chassis: mass 10 -> 10.2035606268
- link left_wheel: mass 1.3542854082 -> 0.15456768270291; geometry collision cylinder length=0.04 radius=0.081; visual mesh filename=package://robot_description/urdf/xlerobot/meshes/xlerobot/a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
- link right_wheel: mass 1.3542854082 -> 0.154567682697732; geometry collision cylinder length=0.04 radius=0.081; visual mesh filename=package://robot_description/urdf/xlerobot/meshes/xlerobot/a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
Joints:
- removed joint ST3215_Servo_Motor-v1-1_Hub-2---Servo
- removed joint ST3215_Servo_Motor-v1-2_Hub---Servo
- removed joint left_wheel_fixed
- removed joint left_wheel_motor_fixed
- removed joint left_wheel_mount_fixed
- removed joint right_wheel_fixed
- removed joint right_wheel_motor_fixed
- removed joint right_wheel_mount_fixed
- removed joint wheel_base_plate_fixed
- added joint left_wheel_drive_joint: type continuous, parent chassis, child left_wheel, origin xyz=-0.002847819 0.265 -0.299 rpy=0 0 0, axis 0 1 0
- added joint right_wheel_drive_joint: type continuous, parent chassis, child right_wheel, origin xyz=-0.002847819 -0.265 -0.299 rpy=0 0 0, axis 0 -1 0

Commit message: feat(simulation): add head RGB camera and ROS image publishing

File: src/robot_description/urdf/xlerobot/xlerobot.urdf (robot description, URDF)
Before this commit: robot xlerobot, 45 links, 44 joints
Joints:
- joint fixed_head_camera_rgb_frame: origin xyz=0 0 0 rpy=0 -1.5707911 -1.5707963 -> xyz=0 0 0 rpy=-1.5707963 0 -1.5707963

Commit message: feat(camera): replace C920 with D415 and add head pan/tilt control

File: src/robot_description/urdf/xlerobot/xlerobot.urdf (robot description, URDF)
Before this commit: robot xlerobot, 45 links, 44 joints
Links:
- removed link world
Joints:
- removed joint joint_0
- joint head_pan_joint: limit lower=-3.2 upper=3.2 effort=0 velocity=0 -> lower=-3.2 upper=3.2 effort=3.35 velocity=2.0
- joint head_tilt_joint: limit lower=-0.76 upper=1.45 effort=0 velocity=0 -> lower=-0.76 upper=1.45 effort=3.35 velocity=2.0
